File: openLRSngTX.brd (EAGLE design)
At the start: 50 x 40 mm, 37 parts, among them IC1 RFM23BPSMD, J1 AVR_SPI_PRG_6PTH, Q1 MMBT2222, U1 ATMEGA328P, X1 BU-SMA-V, Y1 16MHz

Commit message: rev2 modifications
Parts:
- removed C3: 1uF, SparkFun-Capacitors:0805
- removed C9: 10uF, SparkFun-Capacitors:EIA3216
- removed JP4: REG, SparkFun-Connectors:1X03
- added C10: (no value), rcl:D/7343-31W
- added D1: (no value), diode:DO214AC
- added IC2: LT1173CS8, ltc_swr:SOIC8
- added L1: DR74, inductors:DR74
- added R10: 12k, SparkFun-Resistors:0805
- added R11: x, SparkFun-Resistors:0805
- added R9: 270k, SparkFun-Resistors:0805
- S1: device SparkFun-Electromechanical:TACTILE_SWITCH_SMD -> SparkFun-Electromechanical:TACTILE_SWITCH_TALL
- moved C2 7.83 mm to (18.0, 26.0), turned to 0 degrees
- moved R4 4.89 mm to (31.2, 30.5), turned to 180 degrees
- moved R5 4.79 mm to (27.9, 30.5), turned to 0 degrees
- moved R8 3.14 mm to (1.27, 31.2)
- moved R3 2.96 mm to (29.8, 17.5), turned to 270 degrees
- moved LED1 2.36 mm to (31.2, 33.7)
- moved LED2 2.36 mm to (26.7, 33.7)
- moved S1 2.16 mm to (37.2, 33.7), turned to 0 degrees
- moved BIND 2.07 mm to (35.9, 33.5)
- moved C4 1.71 mm to (15.7, 27.4), turned to 270 degrees
- moved R2 1.70 mm to (4.32, 31.2)
- moved R7 0.76 mm to (2.79, 31.2)
- moved C5 0.51 mm to (9.27, 28.2)
- moved Y1 0.38 mm to (12.8, 27.6)
Connections:
- new net N$21: D1.C, IC2.4, L1.1
- new net N$25: IC2.8, R10.2, R11.2, R9.1
- new net VCN: R11.1, U1.11
- net GND: now also C10.-, D1.A, IC2.5, JP1.4, LED1.K, LED2.K, R10.1, S1.B2; no longer C3.2, C9.C, JP1.2, JP4.2, R4.1, R5.1, S1.3
- net N$10: now also LED1.A, R4.1; no longer LED2.K, R5.2
- net N$15: now also S1.A2; no longer S1.1
- net N$17: now also JP1.2; no longer JP1.4
- net N$7: now also R4.2; no longer LED1.A
- net N$8: now also R5.2; no longer LED2.A
- net N$9: now also LED2.A, R5.1; no longer LED1.K, R4.2
- net RAW: now also IC2.1, IC2.2, IC2.3; no longer JP4.1
- net RXD: now also R7.2; no longer R8.2
- net TXD: now also R8.2; no longer R7.2
- net VCC: now also C10.+, L1.2, R9.2; no longer C3.1, C9.A, JP4.3
Routing:
- net N$25: track 0.00 -> 28.8 mm, vias 0 -> 2
- net N$21: track 0.00 -> 19.5 mm
- net VCC: track 133.1 -> 125.1 mm
- net GND: track 10.6 -> 17.0 mm, vias 18 -> 23
- net N$17: track 5.98 -> 11.7 mm
- net N$4: track 15.0 -> 20.4 mm
- net N$15: track 25.9 -> 30.2 mm
- net VCN: track 0.00 -> 2.02 mm
- net N$20: track 6.61 -> 4.79 mm, vias 1 -> 0
- net N$8: track 23.5 -> 25.0 mm, vias 1 -> 2
- net TXD: track 30.4 -> 31.9 mm
- net ICP: track 13.9 -> 15.2 mm
- net N$3: track 9.66 -> 10.6 mm
- net N$11: track 9.14 -> 8.37 mm
- net RXD: track 29.8 -> 30.4 mm
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- removed copper zone on layer 1, net N$16

Commit message: cleaning up
Routing:
- net GND: track 17.0 -> 17.6 mm
Changed lines of the file:
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@@
 <text x="6.223" y="38.354" size="1.016" layer="25">VIN</text>
 <text x="-0.127" y="38.354" size="1.016" layer="25">TXD</text>
-<text x="11.684" y="33.274" size="1.016" layer="25">VCC</text>
-<text x="8.636" y="33.274" size="1.016" layer="25">GND</text>
 <text x="18.034" y="3.556" size="1.016" layer="25" rot="R90">GND</text>
 <text x="20.828" y="3.048" size="1.016" layer="25">SDA</text>
@@
 <text x="9.398" y="2.286" size="1.016" layer="25">SCK</text>
 <text x="12.7" y="2.286" size="1.016" layer="25">RST</text>
-<text x="24.892" y="28.448" size="1.016" layer="26" rot="MR0">GRN</text>
-<text x="29.464" y="28.448" size="1.016" layer="26" rot="MR0">RED</text>
+<text x="28.321" y="30.226" size="1.016" layer="26" rot="MR0">GRN</text>
+<text x="32.766" y="30.226" size="1.016" layer="26" rot="MR0">RED</text>
 <text x="17.78" y="36.322" size="1.27" layer="26" rot="MR180">http://github.com/kh4/openLRSngTX</text>
 <text x="16.256" y="10.414" size="1.016" layer="25">M1</text>
@@
 <element name="J1" library="SparkFun-Connectors" package="2X3" value="AVR_SPI_PRG_6PTH" x="8.255" y="5.08" smashed="yes"/>
 <element name="JP3" library="SparkFun-Connectors" package="1X04" value="I2C" x="19.685" y="5.588" smashed="yes"/>
-<element name="Q1" library="SparkFun-DiscreteSemi" package="SOT23-3" value="MMBT2222" x="32.639" y="17.526" rot="R270"/>
+<element name="Q1" library="SparkFun-DiscreteSemi" package="SOT23-3" value="MMBT2222" x="32.639" y="17.526" smashed="yes" rot="R270">
+<attribute name="NAME" x="32.512" y="17.2085" size="0.4064" layer="25" rot="R270"/>
+<attribute name="VALUE" x="33.7185" y="18.923" size="0.4064" layer="27" rot="R270"/>
+</element>
 <element name="R1" library="SparkFun-Resistors" package="0805" value="10k" x="26.416" y="14.605"/>
 <element name="R2" library="SparkFun-Resistors" package="0805" value="1k" x="4.318" y="31.242" smashed="yes" rot="R270">
@@
 <element name="U$4" library="holes" package="2,8" value="" x="45.72" y="36.322"/>
 <element name="IC2" library="ltc_swr" package="SOIC8" value="LT1173CS8" x="9.271" y="32.004" smashed="yes" rot="R270">
-<attribute name="NAME" x="7.366" y="34.671" size="1.27" layer="25"/>
+<attribute name="NAME" x="8.001" y="29.972" size="1.27" layer="25"/>
 <attribute name="VALUE" x="7.366" y="28.067" size="0.8128" layer="27"/>
 </element>
@@
 <vertex x="-0.635" y="-1.27"/>
 </polygon>
-<wire x1="19.685" y1="25.4" x2="21.209" y2="26.035" width="0.4064" layer="1"/>
+<wire x1="18.934" y1="26.035" x2="21.209" y2="26.035" width="0.4064" layer="1"/>
 <via x="21.209" y="26.035" extent="1-16" drill="0.6"/>
 <via x="17.272" y="11.303" extent="1-16" drill="0.6"/>
@@
 <wire x1="17.018" y1="22.225" x2="17.018" y2="24.257" width="0.4064" layer="1"/>
 <wire x1="17.018" y1="24.257" x2="18.796" y2="26.035" width="0.4064" layer="1"/>
-<wire x1="18.796" y1="26.035" x2="18.934" y2="26.035" width="0.4064" layer="1"/>
+<wire x1="18.796" y1="26.035" x2="18.923" y2="26.035" width="0.4064" layer="1"/>
+<wire x1="18.923" y1="26.035" x2="18.934" y2="26.035" width="0.4064" layer="1"/>
 <wire x1="11.727" y1="28.359" x2="11.727" y2="29.955" width="0.4064" layer="1"/>
 <wire x1="11.727" y1="29.955" x2="11.871" y2="30.099" width="0.4064" layer="1"/>
@@
 <wire x1="15.875" y1="24.765" x2="16.275" y2="24.365" width="0.4064" layer="1"/>
 <wire x1="16.275" y1="24.365" x2="16.275" y2="23.3426" width="0.4064" layer="1"/>
-<wire x1="2.54" y1="17.145" x2="5.715" y2="18.796" width="0.4064" layer="1"/>
-<wire x1="5.715" y1="18.796" x2="7.493" y2="18.796" width="0.4064" layer="1"/>
-<wire x1="7.493" y1="18.796" x2="8.636" y2="18.415" width="0.4064" layer="1"/>
 <via x="8.636" y="18.415" extent="1-16" drill="0.6"/>
 <wire x1="8.636" y1="18.415" x2="10.795" y2="15.24" width="0.4064" layer="16"/>
@@
 <wire x1="17.018" y1="25.919" x2="17.134" y2="26.035" width="0.4064" layer="1"/>
 <wire x1="18.277" y1="27.178" x2="17.134" y2="26.035" width="0.4064" layer="1"/>
+<wire x1="8.636" y1="18.415" x2="5.334" y2="18.415" width="0.4064" layer="1"/>
+<wire x1="5.334" y1="18.415" x2="4.064" y2="17.145" width="0.4064" layer="1"/>
+<wire x1="4.064" y1="17.145" x2="2.54" y2="17.145" width="0.4064" layer="1"/>
 </signal>
 <signal name="RXD">
@@
 <wire x1="21.082" y1="17.907" x2="16.256" y2="17.907" width="0.4064" layer="16"/>
 <via x="16.256" y="17.907" extent="1-16" drill="0.6"/>
-<wire x1="16.256" y1="17.907" x2="15.24" y2="18.415" width="0.4064" layer="1"/>
-<wire x1="15.24" y1="18.415" x2="13.335" y2="20.955" width="0.4064" layer="1"/>
-<wire x1="13.335" y1="20.955" x2="11.6774" y2="20.955" width="0.4064" layer="1"/>
 <wire x1="11.6774" y1="20.955" x2="11.5824" y2="21.05" width="0.4064" layer="1"/>
 <wire x1="30.099" y1="27.051" x2="30.099" y2="27.686" width="0.4064" layer="16"/>
@@
 <wire x1="30.099" y1="27.686" x2="30.099" y2="30.237" width="0.4064" layer="1"/>
 <wire x1="30.099" y1="30.237" x2="30.342" y2="30.48" width="0.4064" layer="1"/>
+<wire x1="11.6774" y1="20.955" x2="13.208" y2="20.955" width="0.4064" layer="1"/>
+<wire x1="13.208" y1="20.955" x2="16.256" y2="17.907" width="0.4064" layer="1"/>
 </signal>
 <signal name="N$8">
 <contactref element="U1" pad="9"/>
-<wire x1="11.5824" y1="21.85" x2="13.71" y2="21.85" width="0.4064" layer="1"/>
-<wire x1="13.71" y1="21.85" x2="13.97" y2="21.59" width="0.4064" layer="1" curve="-90"/>
-<wire x1="13.97" y1="21.59" x2="18.542" y2="18.923" width="0.4064" layer="1"/>
 <via x="18.542" y="18.923" extent="1-16" drill="0.6"/>
 <wire x1="18.542" y1="18.923" x2="20.955" y2="18.923" width="0.4064" layer="16"/>
@@
 <wire x1="28.829" y1="28.956" x2="28.829" y2="30.491" width="0.4064" layer="1"/>
 <wire x1="28.829" y1="30.491" x2="28.84" y2="30.48" width="0.4064" layer="1"/>
+<wire x1="11.5824" y1="21.85" x2="14.599" y2="21.85" width="0.4064" layer="1"/>
+<wire x1="14.599" y1="21.85" x2="17.526" y2="18.923" width="0.4064" layer="1"/>
+<wire x1="17.526" y1="18.923" x2="18.542" y2="18.923" width="0.4064" layer="1"/>
 </signal>
 <signal name="N$11">
@@
 <contactref element="Y1" pad="3"/>
 <wire x1="13.875" y1="23.3426" x2="13.875" y2="24.384" width="0.4064" layer="1"/>
-<wire x1="16.002" y1="28.702" x2="15.748" y2="28.332" width="0.4064" layer="1"/>
 <wire x1="13.875" y1="24.384" x2="12.827" y2="25.908" width="0.254" layer="1"/>
 <wire x1="12.827" y1="25.908" x2="12.827" y2="27.94" width="0.254" layer="1"/>
